Commit message: 控制器初版，控制单个机构位置

File: src/ug_description/urdf/ug_glider.xacro (robot description, xacro)
@@ -10,5 +10,4 @@
   <!-- 引入 UUV Simulator 公共宏 -->
   <xacro:include filename="$(find uuv_descriptions)/urdf/common.urdf.xacro"/>
-  <xacro:include filename="$(find uuv_gazebo_ros_plugins)/urdf/snippets.xacro"/>
   <!-- 引入本模型的各个组件文件，但先不用传感器，用仿真中的真值 -->
   <xacro:include filename="$(find ug_description)/urdf/ug_glider_base.xacro"/>

File: src/ug_description/urdf/ug_glider_actuators.xacro (robot description, xacro)
@@ -1,53 +1,18 @@
 <?xml version="1.0"?>
 <!--
-  水下滑翔机 - 执行器定义 (ros_control 接口)
-  包含：电池滑块传动、方向舵传动
+  水下滑翔机 - 执行器层定义
+  HardwareSimPlugin 直接驱动关节 (SetPosition + preserveWorldVelocity)
+  参考 UUV FinPlugin 的运动学设定方式
 -->
 <robot xmlns:xacro="http://www.ros.org/wiki/xacro">
-  <!-- 引入推进器宏 (必须在宏外部) -->
-  <xacro:include filename="$(find uuv_gazebo_ros_plugins)/urdf/thruster_snippets.xacro"/>
-  <!-- 宏定义  -->
   <xacro:macro name="ug_glider_actuators" params="namespace">
-    <!--电池滑块传动 -->
-    <transmission name="${namespace}/battery_trans">
-      <type>transmission_interface/SimpleTransmission</type>
-      <joint name="${namespace}/battery_joint">
-        <hardwareInterface>hardware_interface/PositionJointInterface</hardwareInterface>
-      </joint>
-      <actuator name="${namespace}/battery_actuator">
-        <mechanicalReduction>1</mechanicalReduction>
-      </actuator>
-    </transmission>
-    <!-- 方向舵传动 (艏摇控制) -->
-    <transmission name="${namespace}/rudder_trans">
-      <type>transmission_interface/SimpleTransmission</type>
-      <joint name="${namespace}/rudder_joint">
-        <hardwareInterface>hardware_interface/PositionJointInterface</hardwareInterface>
-      </joint>
-      <actuator name="${namespace}/rudder_actuator">
-        <mechanicalReduction>1</mechanicalReduction>
-      </actuator>
-    </transmission>
-    <!-- Gazebo ros_control 插件 -->
+    <!-- 硬件抽象仿真插件 -->
     <gazebo>
-      <plugin name="${namespace}_gazebo_ros_control" filename="libgazebo_ros_control.so">
-        <robotNamespace>${namespace}</robotNamespace>
-        <robotSimType>gazebo_ros_control/DefaultRobotHWSim</robotSimType>
-        <legacyModeNS>true</legacyModeNS>
+      <plugin name="${namespace}_hardware_sim" filename="libhardware_sim_plugin.so">
+        <namespace>${namespace}</namespace>
+        <battery_joint>${namespace}/battery_joint</battery_joint>
+        <rudder_joint>${namespace}/rudder_joint</rudder_joint>
       </plugin>
     </gazebo>
-    <!-- 浮力系统 (VBS控制) -->
-    <!-- 已迁移到 ug_glider_gazebo.xacro 中的 libbuoyancy_engine_plugin.so -->
-    <!-- 基于物理的油囊模型，通过控制体积产生浮力差 -->
-    <!-- 推进器等效浮力方案 -->
-    <!-- 用一个垂直螺旋桨的力来等效浮力，控制律需要映射节点 -->
-    <!-- <xacro:thruster_module_first_order_basic_fcn_macro
-      namespace="${namespace}"
-      thruster_id="0"
-      mesh_filename="package://ug_description/meshes/ug_oil.stl"
-      dyn_time_constant="0.5"
-      rotor_constant="10.08">
-      <origin xyz="-0.361 0 -0.052" rpy="0 ${-pi/2} 0"/>
-    </xacro:thruster_module_first_order_basic_fcn_macro> -->
   </xacro:macro>
 </robot>

File: src/ug_description/urdf/ug_glider_base.xacro (robot description, xacro)
@@ -12,5 +12,5 @@
   <!-- 参数定义  -->
   <!-- 船体参数 -->
-  <xacro:property name="hull_mass" value="20.26"/>           <!-- 干重 [kg]，目前假设质量等于（体积-500cc）*海水密度-舵-固定翼（assume） -->
+  <xacro:property name="hull_mass" value="24.485"/>           <!-- 干重 [kg]，目前假设质量等于（体积-500cc）*海水密度-舵-固定翼（assume） -->
   <xacro:property name="hull_length" value="1.252"/>          <!-- 总长度 [m] -->
   <xacro:property name="hull_diameter" value="0.255"/>       <!-- 船体直径 [m] -->
@@ -28,12 +28,12 @@
   <!-- 电池滑块参数-->  <!--注意现在配平尚有问题-->
   <xacro:property name="battery_mass" value="10.0"/>        <!-- assume的电池包质量 [kg] -->
-  <xacro:property name="battery_travel" value="0.012"/>      <!-- 最大行程半径 [m] -->
-  <xacro:property name="battery_x_origin" value="-0.1115"/>     <!-- 电池中立位置 [m]-0.12385 -->
+  <xacro:property name="battery_travel" value="0.03385"/>      <!-- 最大行程半径 [m] -->
+  <xacro:property name="battery_x_origin" value="0.0"/>     <!-- 先assume电池质心与hull质心重合，-0.1115电池中立位置 [m]-0.12385 -->
   <!--暂时值，目前与800cc配平-->
   <!-- 方向舵参数 -->
-  <xacro:property name="rudder_mass" value="0.225"/>          <!-- 舵质量 [kg] -->
+  <xacro:property name="rudder_mass" value="1.0e-6"/>          <!-- 舵质量都在hull里，为了浮力和重力统一，避免冗余力矩 -->
   <xacro:property name="rudder_max_angle" value="0.52"/>    <!-- assume最大偏转角 [rad] (~30度) -->
   <!-- 固定翼参数 -->
-  <xacro:property name="wing_mass" value="4.0"/>            <!-- assume翼组件质量 [kg] -->
+  <xacro:property name="wing_mass" value="1.0e-6"/>            <!-- 翼组件质量都在hull里，为了浮力和重力统一，避免冗余力矩 -->
   <xacro:property name="wing_x" value="-0.325"/>            <!-- 翼位置X [m] -->
   <xacro:property name="wing_z" value="0.15"/>              <!-- 翼位置Z [m] -->
@@ -88,5 +88,5 @@
         <origin xyz="0 0 0" rpy="0 0 0"/>
         <geometry>
-          <box size="0.3 0.1 0.08"/>
+          <box size="0.03 0.01 0.008"/>
         </geometry>
       </collision>
@@ -95,5 +95,5 @@
       <parent link="${namespace}/base_link"/>
       <child link="${namespace}/battery_link"/>
-      <origin xyz="${battery_x_origin} 0 0" rpy="0 0 0"/>
+      <origin xyz="${battery_x_origin} 0 -0.05" rpy="0 0 0"/>  <!-- assume电池z向质心与hull一样 -->
       <axis xyz="1 0 0"/>  <!-- 沿X轴滑动 (前后方向)，后续再添加roll控制 -->
       <limit lower="${-battery_travel}" upper="${battery_travel}" effort="100" velocity="0.05"/>

File: src/ug_description/urdf/ug_glider_gazebo.xacro (robot description, xacro)
@@ -10,5 +10,5 @@
   <xacro:property name="fluid_density" value="1028.0"/>     <!-- 海水密度 [kg/m^3] -->
   <!-- 浮力参数 -->
-  <xacro:property name="hull_volume" value="0.0336"/>        <!-- 排水体积，扣除500cc油馕体积 [m^3] -->
+  <xacro:property name="hull_volume" value="0.033547"/>       <!-- 排水体积 [m^3]，由 total_mass/fluid_density = 34.486/1028 得出，确保中性油量时零净浮力 -->
   <xacro:property name="cob_x" value="0.0"/>                <!-- 浮心位置 (原点) -->
   <xacro:property name="cob_y" value="0.0"/>
@@ -18,5 +18,5 @@
   <xacro:property name="oil_min_volume" value="0.0"/>           <!-- 油囊最小体积 0cc [m^3] -->
   <xacro:property name="oil_max_volume" value="0.001"/>         <!-- 油囊最大体积 1000cc [m^3] -->
-  <xacro:property name="oil_pump_rate" value="0.0001"/>         <!-- 油泵流速 100cc/s [m^3/s] -->
+  <!-- 油泵流速已移至 ug_hardware_sim 参数配置 -->
   <xacro:property name="oil_bladder_x" value="-0.361"/>         <!-- 油囊位置x（尾部）[m] -->
   <xacro:property name="oil_bladder_y" value="-0.0005"/>        <!-- 油囊位置y [m] -->
@@ -159,11 +159,9 @@
         <min_volume>${oil_min_volume}</min_volume>
         <max_volume>${oil_max_volume}</max_volume>
-        <initial_volume>0.0008</initial_volume>  <!-- 启动时油囊初始体积 500cc -->
-        <!-- 油泵动态 -->
-        <pump_rate>${oil_pump_rate}</pump_rate>
+        <initial_volume>0.0005</initial_volume>  <!-- 启动时油囊初始体积 500cc -->
         <!-- 油囊力作用点（相对于base_link，产生俯仰力矩）-->
         <bladder_position>${oil_bladder_x} ${oil_bladder_y} ${oil_bladder_z}</bladder_position>
-        <!-- ROS话题 -->
-        <command_topic>buoyancy_engine/cmd_volume</command_topic>
+        <!-- ROS话题（接收 ug_hardware_sim 发布的实际体积）-->
+        <command_topic>buoyancy_engine/set_volume</command_topic>
         <status_topic>buoyancy_engine/status</status_topic>
       </plugin>
