Commit message: 电池滚转控制

File: src/glider_sim/ug_description/urdf/ug_glider_actuators.xacro (robot description, xacro)
@@ -12,4 +12,5 @@
         <namespace>${namespace}</namespace>
         <battery_joint>${namespace}/battery_joint</battery_joint>
+        <battery_roll_joint>${namespace}/battery_roll_joint</battery_roll_joint>
         <rudder_joint>${namespace}/rudder_joint</rudder_joint>
       </plugin>

File: src/glider_sim/ug_description/urdf/ug_glider_base.xacro (robot description, xacro)
@@ -67,12 +67,28 @@
       </inertial>
     </link>
-    <!-- 电池滑块，目前只能前后移动 -->
+    <!-- 电池滑块（虚拟中间 link，仅用于串联 prismatic + revolute 两个自由度） -->
+    <link name="${namespace}/battery_slide_link">
+      <inertial>
+        <mass value="1e-6"/>
+        <origin xyz="0 0 0" rpy="0 0 0"/>
+        <inertia ixx="1e-8" ixy="0" ixz="0" iyy="1e-8" iyz="0" izz="1e-8"/>
+      </inertial>
+    </link>
+    <!-- 电池前后平移，控制 pitch -->
+    <joint name="${namespace}/battery_joint" type="prismatic">
+      <parent link="${namespace}/base_link"/>
+      <child link="${namespace}/battery_slide_link"/>
+      <origin xyz="${battery_x_origin} 0 -0.05" rpy="0 0 0"/>
+      <axis xyz="1 0 0"/>
+      <limit lower="${-battery_travel}" upper="${battery_travel}" effort="100" velocity="0.05"/>
+      <dynamics damping="10.0" friction="1.0"/>
+    </joint>
+    <!-- 电池本体，质心偏离旋转轴 0.03m（向下），旋转时质心侧移产生 roll 力矩 -->
     <link name="${namespace}/battery_link">
       <inertial>
         <mass value="${battery_mass}"/>
-        <origin xyz="0 0 0" rpy="0 0 0"/>
+        <origin xyz="0 0 -0.03" rpy="0 0 0"/>
         <inertia ixx="0.01" ixy="0" ixz="0" iyy="0.01" iyz="0" izz="0.01"/>
       </inertial>
-      <!-- 调试用可视化 (小方块表示电池包) -->
       <visual>
         <origin xyz="0 0 0" rpy="0 0 0"/>
@@ -91,11 +107,12 @@
       </collision>
     </link>
-    <joint name="${namespace}/battery_joint" type="prismatic">
-      <parent link="${namespace}/base_link"/>
+    <!-- 电池绕纵轴旋转，控制 roll -->
+    <joint name="${namespace}/battery_roll_joint" type="revolute">
+      <parent link="${namespace}/battery_slide_link"/>
       <child link="${namespace}/battery_link"/>
-      <origin xyz="${battery_x_origin} 0 -0.05" rpy="0 0 0"/>  <!-- assume电池z向质心与hull一样 -->
-      <axis xyz="1 0 0"/>  <!-- 沿X轴滑动 (前后方向)，后续再添加roll控制 -->
-      <limit lower="${-battery_travel}" upper="${battery_travel}" effort="100" velocity="0.05"/>
-      <dynamics damping="10.0" friction="1.0"/>
+      <origin xyz="0 0 0" rpy="0 0 0"/>
+      <axis xyz="1 0 0"/>
+      <limit lower="-1.57" upper="1.57" effort="50" velocity="1.0"/>
+      <dynamics damping="0.5" friction="0.1"/>
     </joint>
     <!-- 尾舵  -->

File: src/glider_sim/ug_description/urdf/ug_glider_gazebo.xacro (robot description, xacro)
@@ -5,4 +5,5 @@
   uuv_sim的fin插件不适配Gazebo 11，目前使用Gazebo自带插件，后续自己开发，这个已经实现，固定翼和转向舵都挂载升阻力插件
 -->
+<!--为演示，尾舵cp挂载在z=质心，这样roll就可以暂不处理，后续再处理-->
 <robot xmlns:xacro="http://www.ros.org/wiki/xacro">
   <!-- 水动力参数 (TODO: 填入实际数据) -->
@@ -150,5 +151,5 @@
         <fluid_density>${fluid_density}</fluid_density>
         <area>${rudder_area}</area>
-        <cp>-0.417 0 0.09</cp>
+        <cp>-0.417 0 -0.05</cp><!--为演示，尾舵z位置质心，这样roll就可以暂不处理，后续再处理-->
         <forward>1 0 0</forward>
         <upward>0 1 0</upward>
@@ -166,10 +167,10 @@
     <!-- 分层洋流插件 -->
     <!-- 根据滑翔机深度实时插值洋流，同时发布到 Gazebo transport用于物理计算和 ROS用于调试 -->
-    <!-- 数据源：SDF <layer> 标签（简单模式）或 CS  <!-- 简单模式：ENU 分层表 (vx=东, vy=北, vz=上) -->
+    <!-- 数据源：SDF <layer> 标签（简单模式）或 简单模式：ENU 分层表 (vx=东, vy=北, vz=上) -->
         <layer depth="0"   vx="0.1"  vy="0.0" vz="0.0"/>
         <layer depth="10"  vx="0.08" vy="0.0" vz="0.0"/>
         <layer depth="20"  vx="0.03" vy="0.0" vz="0.0"/>
         <layer depth="30"  vx="0.0"  vy="0.0" vz="0.0"/>
-V 文件（真实海洋数据模式），CSV是DAVE开发用到的格式，要有个脚本把CFD数据转成CSV -->
+<!--文件（真实海洋数据模式），CSV是DAVE开发用到的格式，要有个脚本把CFD数据转成CSV -->
     <gazebo>
       <plugin name="${namespace}_ocean_current" filename="libug_ocean_current_plugin.so">
