Commit message: Swarm Version 1

File: src/glider_sim/ug_description/urdf/ug_glider.xacro (robot description, xacro)
@@ -8,4 +8,5 @@
   <xacro:arg name="debug" default="0"/>
   <xacro:arg name="namespace" default="ug_glider"/>
+  <xacro:arg name="hull_color" default="Yellow"/>
   <!-- 引入 UUV Simulator 公共宏 -->
   <xacro:include filename="$(find uuv_descriptions)/urdf/common.urdf.xacro"/>
@@ -16,5 +17,5 @@
   <!-- 实例化滑翔机各组件 -->
   <xacro:ug_glider_base namespace="$(arg namespace)"/>
-  <xacro:ug_glider_gazebo namespace="$(arg namespace)" debug="$(arg debug)"/>
+  <xacro:ug_glider_gazebo namespace="$(arg namespace)" debug="$(arg debug)" hull_color="$(arg hull_color)"/>
   <xacro:ug_glider_actuators namespace="$(arg namespace)"/>
 </robot>

File: src/glider_sim/ug_description/urdf/ug_glider_gazebo.xacro (robot description, xacro)
@@ -57,5 +57,5 @@
   <xacro:property name="rudder_drag_coef" value="0.017"/>     <!-- 阻力系数 -->
   <!-- 宏定义 -->
-  <xacro:macro name="ug_glider_gazebo" params="namespace debug">
+  <xacro:macro name="ug_glider_gazebo" params="namespace debug hull_color:=Yellow">
     <!-- 水下插件 (Fossen水动力模型) -->
     <gazebo>
@@ -168,7 +168,7 @@
     <!-- 根据滑翔机深度实时插值洋流，同时发布到 Gazebo transport用于物理计算和 ROS用于调试 -->
     <!-- 数据源：SDF <layer> 标签（简单模式）或 简单模式：ENU 分层表 (vx=东, vy=北, vz=上) -->
-        <layer depth="0"   vx="0.1"  vy="0.0" vz="0.0"/>
-        <layer depth="10"  vx="0.08" vy="0.0" vz="0.0"/>
-        <layer depth="20"  vx="0.03" vy="0.0" vz="0.0"/>
+        <layer depth="0"   vx="0.0"  vy="0.0" vz="0.0"/>
+        <layer depth="10"  vx="0.0" vy="0.0" vz="0.0"/>
+        <layer depth="20"  vx="0.0" vy="0.0" vz="0.0"/>
         <layer depth="30"  vx="0.0"  vy="0.0" vz="0.0"/>
 <!--文件（真实海洋数据模式），CSV是DAVE开发用到的格式，要有个脚本把CFD数据转成CSV -->
@@ -210,5 +210,5 @@
     <!-- Gazebo 材质颜色 -->
     <gazebo reference="${namespace}/base_link">
-      <material>Gazebo/Yellow</material>
+      <material>Gazebo/${hull_color}</material>
     </gazebo>
     <gazebo reference="${namespace}/rudder_link">

Commit message: Swarm以及Communacation

File: src/glider_sim/ug_description/urdf/ug_glider.xacro (robot description, xacro)
@@ -9,4 +9,5 @@
   <xacro:arg name="namespace" default="ug_glider"/>
   <xacro:arg name="hull_color" default="Yellow"/>
+  <xacro:arg name="hull_rgba" default="1.0 0.9 0.0 1.0"/>
   <!-- 引入 UUV Simulator 公共宏 -->
   <xacro:include filename="$(find uuv_descriptions)/urdf/common.urdf.xacro"/>
@@ -16,5 +17,5 @@
   <xacro:include filename="$(find ug_description)/urdf/ug_glider_actuators.xacro"/>
   <!-- 实例化滑翔机各组件 -->
-  <xacro:ug_glider_base namespace="$(arg namespace)"/>
+  <xacro:ug_glider_base namespace="$(arg namespace)" hull_rgba="$(arg hull_rgba)"/>
   <xacro:ug_glider_gazebo namespace="$(arg namespace)" debug="$(arg debug)" hull_color="$(arg hull_color)"/>
   <xacro:ug_glider_actuators namespace="$(arg namespace)"/>

File: src/glider_sim/ug_description/urdf/ug_glider_base.xacro (robot description, xacro)
@@ -41,5 +41,5 @@
   <xacro:property name="rudder_mesh" value="package://ug_description/meshes/UG_steer.stl"/>
   <!-- 宏定义 -->
-  <xacro:macro name="ug_glider_base" params="namespace">
+  <xacro:macro name="ug_glider_base" params="namespace hull_rgba:='1.0 0.9 0.0 1.0'">
     <!-- 机体 (base_link)-->
     <link name="${namespace}/base_link">
@@ -49,6 +49,6 @@
           <mesh filename="${hull_mesh}" scale="1 1 1"/>
         </geometry>
-        <material name="glider_yellow">
-          <color rgba="1.0 0.9 0.0 1.0"/>
+        <material name="${namespace}_hull_material">
+          <color rgba="${hull_rgba}"/>
         </material>
       </visual>
